File: hardware/kicad/open-hardware-wallet-v1/open-hardware-wallet-v1.kicad_sch (KiCad schematic)
At the start: 6 parts, among them J1 USB_C_Receptacle_PowerOnly_6P

Commit message: Add power input and LDO schematic draft
Parts:
- added C1, C3: 10uF, C0603, symbol Device:C
- added C2: 100uF, CAP-SMD_L3.2-W1.6, symbol Device:C_Polarized
- added C4: 100nF, C0402, symbol Device:C
- added D4: 1N5819W, Diode_SMD:D_SOD-323, symbol Diode:1N5819WS
- added Q1: SI2301ADS-T1-GE3-VB, symbol Transistor_FET:Q_PMOS_GSD
- added R3: 100kΩ, R0402, symbol Device:R
- added R4: 10kΩ, R0402, symbol Device:R
- added U1: AP2112K-3.3TRG1, Package_TO_SOT_SMD:SOT-23-5, symbol Regulator_Linear:AP2112K-3.3
Connections:
- net GND: now also C1.2, C2.2, C3.2, C4.2, R3.1, U1.2 (GND)
- net VBUS: now also D4.2 (A), Q1.1 (G), R3.2
- new net: R4.1, U1.3 (EN)
- new net: C1.1, D4.1 (K), Q1.2 (S), R4.2, U1.1 (VIN)
- new net +3V3: C2.1, C3.1, C4.1, U1.5 (VOUT)
Other:
- note added: "USB-C Power Input & Protection"
- note added: "VBUS / VBAT to 3.3V LDO Regulator"
- note removed: "USB_C_POWER"

Commit message: Add Stage 2: Battery Charging, Voltage Monitoring & SPI Flash documentation and schematics
Parts:
- added C5: 10uF, C0603, symbol Device:C
- added C6: 100nF, C0402, symbol Device:C
- added R10, R11, R9: 10kΩ, R0402, symbol Device:R
- added R5: 4.7kΩ, R0603, symbol Device:R
- added R6: 2.2kΩ, R0402, symbol Device:R
- added R7, R8: 100kΩ, R0402, symbol Device:R
- added U2: MCP73831T-2DCI/OT, Package_TO_SOT_SMD:SOT-23-5, symbol Battery_Management:MCP73831-2-OT
- added U3: W25Q64JVZPIQ, Package_SON:WSON-8-1EP_6x5mm_P1.27mm_EP3.4x4.3mm, symbol Memory_Flash:W25Q32JVZP
Connections:
- net +3V3: now also R10.2, R11.2, R6.2, R9.1
- net GND: now also C6.2, R5.1, R8.1, U3.4 (GND), U3.9 (EP)
- net VBUS: now also U2.4 (V_{DD})
- net VBAT: now reaches Q1.3 (D)
- net VBAT: now also C5.1, R7.2, U2.3 (V_{BAT})
- new net: C5.2, U2.2 (V_{SS})
- new net: R5.2, U2.5 (PROG)
- new net: R10.1, U3.3 (~{WP}/IO_{2})
- new net: R11.1, U3.7 (~{HOLD}/~{RESET}/IO_{3})
- new net BAT_ADC: C6.1, R7.1, R8.2
- new net BAT_STAT: R6.1, U2.1 (STAT)
- new net FLASH_CLK: U3.6 (CLK)
- new net FLASH_CS#: R9.2, U3.1 (~{CS})
- new net FLASH_MISO: U3.2 (DO/IO_{1})
- new net FLASH_MOSI: U3.5 (DI/IO_{0})
Other:
- note added: "Battery Voltage Monitoring"
- note added: "External SPI Flash Memory"
- note added: "Ireg = 1000 / Rprog [kΩ] unit: mA =210mA"
- note added: "Li-ion Battery Charging"
- moved on the sheet: C1, C2, C3, C4, D4, Q1, R3, R4, U1

Commit message: Update project progress: Step3–Step5 documentation and PCB schematic updates
Parts:
- added C10, C12, C15, C17, C18, C23, C25, C27, C29, C34, C7, C8, C9: 1uF, C0402, symbol Device:C
- added C11, C14, C16, C22, C24, C26, C28, C32, C33: 100nF, C0402, symbol Device:C
- added C13: 10uF, C0603, symbol Device:C
- added C19: 4.7uF, C0402, symbol Device:C
- added C20: 2.2uF, C0402, symbol Device:C
- added C21: 4.7uF, C0603, symbol Device:C
- added C30: 18F, C0402, symbol Device:C
- added C31: 18pF, C0402, symbol Device:C
- added D5, D6: LED, symbol Device:LED
- added D7: 1N4148WS, Diode_SMD:D_SOD-323, symbol Diode:1N4148WS
- added DS1: OLED-128O064D-FPC-30P, Display:OLED-128O064D, symbol Havenlon_Symbol_Connector:OLED-128O064D-FPC-30P
- added FID1, FID2, FID3: Fiducial, symbol Mechanical:Fiducial
- added H1, H2, H3, H4: MountingHole_Pad, symbol Mechanical:MountingHole_Pad
- added IC1: SE050E2HQ1, QFN40P300X300X33-21N-D, symbol Havenlon_Symbol_IC:SE050E2HQ1
- added J2: Conn_01x08_Pin, symbol Connector:Conn_01x08_Pin
- added L1: L, symbol Device:L
- added R12, R13, R14, R15, R18, R19, R27, R28, R29: 10kΩ, R0402, symbol Device:R
- added R16, R17: 47Ω, R0402, symbol Device:R
- added R20, R21, R22, R23, R25: 4.7kΩ, R0402, symbol Device:R
- added R24: 620kΩ, R0402, symbol Device:R
- added R26: 0Ω, R0402, symbol Device:R
- added SW1, SW2, SW3, SW4: KH-4.5X4.5X4.3H-STM, symbol Switch:SW_MEC_5E
- added TP1, TP2, TP3, TP4: TestPoint, symbol Connector:TestPoint
- added U4: EWM104-BT09SP, symbol Havenlon_Symbol_Module:BT_Module_EWM104_BT09SP
- added U6: STM32L476RET6, Package_QFP:LQFP-64_10x10mm_P0.5mm, symbol Havenlon_Symbol_IC:STM32L476RET6
- added Y1: Crystal-8M, symbol Device:Crystal
Connections:
- net +3V3: now also C11.1, C12.1, C13.1, C14.1, C15.1, C16.1, C22.1, C23.1, C24.1, C25.1, C26.1, C27.1, C28.1, C29.1, D5.2 (A), D6.2 (A), D7.1 (K), DS1.11 (BS1), DS1.6 (VBAT), DS1.9 (VDD), IC1.12 (VIN), IC1.13 (ISO_7816_CLK), IC1.17 (ISO_14443_LA), IC1.18 (VCC), IC1.3 (ISO_7816_IO1), J2.5 (Pin_5), L1.1, R12.1, R13.1, R14.1, R15.1, R20.1, R21.2, R22.1, R23.1, R25.1, R26.2, R28.1, TP2.1, U4.12 (VBAT), U6.19 (VDD), U6.32 (VDD), U6.48 (VDDUSB), U6.64 (VDD)
- net BAT_ADC: now also U6.15 (PA1)
- net BAT_STAT: now also U6.56 (PB4)
- net FLASH_CLK: now also U6.21 (PA5)
- net FLASH_CS#: now also U6.17 (PA3)
- net FLASH_MISO: now also U6.22 (PA6)
- net FLASH_MOSI: now also U6.23 (PA7)
- net GND: now also C10.2, C11.2, C12.2, C13.2, C14.2, C15.2, C16.2, C19.2, C20.1, C21.1, C22.2, C23.2, C24.2, C25.2, C26.2, C27.2, C28.2, C29.2, C30.2, C31.2, C32.2, C33.2, C34.2, C7.2, C8.2, C9.2, DS1.1 (GND), DS1.10 (BS0), DS1.12 (BS2), DS1.13 (~{CS}), DS1.15 (D/~{C}), DS1.16 (R/~{W}), DS1.17 (E/~{RD}), DS1.21 (D3), DS1.22 (D4), DS1.23 (D5), DS1.24 (D6), DS1.25 (D7), DS1.29 (VLSS), DS1.30 (GND), DS1.8 (VSS), H1.1, H2.1, H3.1, H4.1, IC1.1 (ISO_14443_LB), IC1.19 (VSS), IC1.21 (EP), J2.4 (Pin_4), J2.8 (Pin_8), R18.1, R24.1, R27.1, R29.1, SW1.3 (K), SW1.4 (A), SW2.3 (K), SW2.4 (A), SW3.3 (K), SW3.4 (A), SW4.3 (K), SW4.4 (A), TP4.1, U4.1 (GND), U4.11 (GND), U4.18 (GND), U6.18 (VSS), U6.31 (VSS), U6.47 (VSS), U6.63 (VSS)
- new net: D5.1 (K), R18.2
- new net: C17.1, DS1.2 (C2N)
- new net: DS1.26 (IREF), R24.2
- new net: C19.1, DS1.27 (VCOMH)
- new net: C20.2, DS1.28 (VCC)
- new net: C17.2, DS1.3 (C2P)
- new net: C18.1, DS1.4 (C1P)
- new net: C18.2, DS1.5 (C1N)
- new net: C21.2, D7.2 (A), R25.2
- new net: R16.1, U4.9 (RXD)
- new net: R17.2, U4.10 (TXD)
- new net: D6.1 (K), R19.1
- new net: C30.1, Y1.1
- new net: R26.1, U6.1 (VBAT)
- new net: C31.1, Y1.2
- new net BOOT0: R27.2, TP1.1, U6.60 (BOOT0)
- new net BT_LINK: U4.5 (PA7), U6.50 (PA15)
- new net BT_RX: R16.2, U6.24 (PC4)
- new net BT_TX: R17.1, U6.25 (PC5)
- new net BT_WKP: U4.8 (WKP), U6.26 (PB0)
- new net DBG_RX: J2.3 (Pin_3), U6.43 (PA10)
- new net DBG_TX: J2.2 (Pin_2), U6.42 (PA9)
- new net GNDA: R29.2, U6.12 (VSSA)
- new net K_CANCEL: C7.1, R12.2, SW1.1, SW1.2, U6.40 (PC9)
- new net K_DOWN: C9.1, R14.2, SW3.1, SW3.2, U6.38 (PC7)
- new net K_OK: C10.1, R15.2, SW4.1, SW4.2, U6.37 (PC6)
- new net K_UP: C8.1, R13.2, SW2.1, SW2.2, U6.39 (PC8)
- new net LED: R19.2, U6.2 (PC13)
- new net NRST: C32.1, J2.1 (Pin_1), R28.2, TP3.1, U6.7 (NRST)
- new net OLED_SCL: DS1.18 (D0), R22.2, U6.58 (PB6)
- new net OLED_SDA: DS1.19 (D1), DS1.20 (D2), R23.2, U6.59 (PB7)
- new net OSCIN: U6.3 (PC14)
- new net OSCOUT: U6.4 (PC15)
- new net RES#: DS1.14 (~{RES})
- new net SE05_ENA: IC1.11 (ENA), U6.27 (PB1)
- new net SE05_SCL: IC1.10 (L2C_SCL), R21.1, U6.29 (PB10)
- new net SE05_SDA: IC1.9 (L2C_SDA), R20.2, U6.30 (PB11)
- new net SWDCLK: J2.6 (Pin_6), U6.49 (PA14)
- new net SWDDIO: U6.46 (PA13)
- new net SWDIO: J2.7 (Pin_7)
- new net VDDA: C33.1, C34.1, L1.2, U6.13 (VDDA)
- no-connect marks 0 -> 48
Other:
- note added: "Analog Power Filter"
- note added: "Bluetooth Module Interface"
- note added: "Boot"
- note added: "Crystal oscillator: 8 MHz"
- note added: "Debug"
- note added: "Decoupling capacitors"
- note added: "MCU: STM32L476RET6"
- note added: "Mechanical Mounting & Fiducials"
- note added: "NRST"
- note added: "OLED 13XX Display Interface"
- note added: "Power & Status LEDs"
- note added: "SE05X Secure Element Interface"
- note added: "User Input Keypad / Navigation Buttons"
- company: (none) -> Havenlon
- title: (none) -> Havenlon Open Hardware Wallet V1
